File: Project-Aurora.sch (KiCad schematic (older format))
At the start: 62 parts, among them P1 USB_OTG, P10 DBG, P11 DBG, P12 DBG, P2 FLASH_HDR, P3 DBG, P4 DBG, P5 DBG, P6 DBG, P7 DBG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

Commit message: Switched to a different USB Port and 100uF Cap
also added a USB-Debug Header and did some cleanup
Parts:
- added P13: CONN_01X04, Pin_Headers:Pin_Header_Straight_1x04_Pitch2.00mm, symbol CONN_01X04
- C20: footprint Capacitors_SMD:C_0805 -> Capacitors_SMD:C_1206
- P1: footprint Connect:USB_Micro-B -> libs.pretty:Micro-USB_629105150521
Connections:
- net labels added: D+5V, D-5V
